Commit message: Added robot state publisher and rgb camera

File: box_bot_description/robot/box_bot.urdf (robot description, URDF)
Before this commit: robot box_bot, 10 links, 9 joints
Links:
- added link rgb_cam_camera_link; visual box size=0.01 0.01 0.01
- added link rgb_cam_camera_link_frame
Joints:
- added joint rgb_cam_camera_frame_joint: type fixed, parent rgb_cam_camera_link, child rgb_cam_camera_link_frame, origin xyz=0.01 0 0 rpy=0 0 0, axis 0 0 0
- added joint rgb_cam_camera_link_joint: type fixed, parent chassis, child rgb_cam_camera_link, origin xyz=0.04 0.0 0.045 rpy=0 0 0

File: box_bot_description/robot/box_bot_v2.urdf (robot description, URDF)
Before this commit: robot box_bot, 10 links, 9 joints
Links:
- added link rgb_cam_camera_link; visual box size=0.01 0.01 0.01
- added link rgb_cam_camera_link_frame
Joints:
- added joint rgb_cam_camera_frame_joint: type fixed, parent rgb_cam_camera_link, child rgb_cam_camera_link_frame, origin xyz=0.01 0 0 rpy=0 0 0, axis 0 0 0
- added joint rgb_cam_camera_link_joint: type fixed, parent chassis, child rgb_cam_camera_link, origin xyz=0.04 0.0 0.045 rpy=0 0 0
