Commit message: Added pointcloud

File: box_bot_description/robot/box_bot_with_meshes.xacro (robot description, xacro)
@@ -16,5 +16,6 @@
   <xacro:caster_wheel parent="chassis" caster_wheel_name="front" origin_xyz="${(base_box_x / 2.0) - wheel_increment} 0 ${-1.0* base_box_x / 2.0}" radius="${wheel_increment}" legth="${dummy_length}"/>
   <xacro:caster_wheel parent="chassis" caster_wheel_name="back" origin_xyz="${(-1.0 *base_box_x / 2.0) + wheel_increment} 0 ${-1.0* base_box_x / 2.0}" radius="${wheel_increment}" legth="${dummy_length}"/>
-  <xacro:camera_rgb parent_name="${base_name}" sensor_name="rgb_camera" origin_xyz="${base_box_x} 0.0 ${base_box_x / 2.0}" camera_ROLL="0.0" camera_PITCH="0.0" camera_YAW="0.0"/>
+  <xacro:camera_rgb parent_name="${base_name}" sensor_name="rgb_camera" origin_xyz="${base_box_x/ 1.9} 0.0 ${base_box_x / 2.0}" camera_ROLL="0.0" camera_PITCH="0.0" camera_YAW="0.0"/>
   <xacro:laser_scan parent_name="${base_name}" sensor_name="laser_scan" origin_xyz="0.0 0.0 ${base_box_x / 1.5}" sensor_YAW="1.57"/>
+  <xacro:block_laser_scan parent_name="${base_name}" sensor_name="block_laser_scan" origin_xyz="${base_box_x/ 1.9} 0.0 ${base_box_x / 2.0}" sensor_YAW="1.57"/>
 </robot>

File: box_bot_description/robot/sensors.xacro (robot description, xacro)
@@ -7,5 +7,6 @@
 					rpy="0 0 0"/>
 			<geometry>
-				<box size="${camera_box_x} ${camera_box_y} ${camera_box_z}"/>
+				<!-- <box size="${camera_box_x} ${camera_box_y} ${camera_box_z}"/> -->
+                 <mesh filename="package://box_bot_description/meshes/sensors/realsense.dae" scale="0.25 0.25 0.25"/>
 			</geometry>
 		</visual>
@@ -137,5 +138,5 @@
         <visual name="visual_${parent_name}">
             <geometry>
-                    <mesh filename="package://box_bot_description/meshes/sensors/rplidar.dae" scale="${base_box_x} ${base_box_y} ${base_box_z}"/>
+                    <mesh filename="package://box_bot_description/meshes/sensors/rplidar.dae" scale="1.0 1.0 1.0"/>
             </geometry>
         </visual>
@@ -184,3 +185,70 @@
 	</gazebo>
   </xacro:macro>
+<xacro:macro name="block_laser_scan" params="parent_name sensor_name origin_xyz sensor_YAW">
+    <link name='${sensor_name}_laser_scan_link'>
+        <visual name="visual_${parent_name}">
+            <geometry>
+                    <mesh filename="package://box_bot_description/meshes/sensors/realsense.dae" scale="0.25 0.25 0.25"/>
+            </geometry>
+        </visual>
+	</link>
+    <joint name="${sensor_name}_laser_scan_link_joint" type="fixed">
+		<origin rpy="0 0 ${sensor_YAW - 1.5708}" xyz="${origin_xyz}"/>
+		<parent link="${parent_name}"/>
+		<child link="${sensor_name}_laser_scan_link"/>
+	</joint>
+    <link name="${sensor_name}_laser_scan_frame">
+    </link>
+    <joint name="${sensor_name}_laser_scan_frame_joint" type="fixed">
+        <origin xyz="0 0 0" rpy="0 0 0" />
+        <parent link="${sensor_name}_laser_scan_link" />
+        <child link="${sensor_name}_laser_scan_frame" />
+        <axis xyz="0 0 0"/>
+    </joint>
+    <gazebo reference="${sensor_name}_laser_scan_frame">
+        <sensor type="ray" name="block_laser_sensor">
+            <ray>
+            <scan>
+                <horizontal>
+                    <samples>50</samples>
+                    <resolution>1.0</resolution>
+                    <min_angle>-1.0</min_angle>
+                    <max_angle>1.0</max_angle>
+                </horizontal>
+                <vertical>
+                    <samples>50</samples>
+                    <resolution>1.0</resolution>
+                    <min_angle>-1.0</min_angle>
+                    <max_angle>1.0</max_angle>
+                </vertical>
+            </scan>
+            <range>
+                <min>0.10</min>
+                <max>5.0</max>
+                <resolution>0.01</resolution>
+            </range>
+            <!-- Using gazebo's noise instead of plugin's -->
+            <noise>
+                <type>gaussian</type>
+                <mean>0.0</mean>
+                <stddev>0.01</stddev>
+            </noise>
+            </ray>
+            <!-- Using gazebo's update rate instead of plugin's -->
+            <update_rate>30</update_rate>
+            <plugin name="gazebo_ros_block_laser_controller" filename="libgazebo_ros_ray_sensor.so">
+            <!-- Change namespace and output topic so published topic is /rrbot/laser/pointcloud -->
+            <ros>
+                <namespace>/rrbot/laser</namespace>
+                <argument>~/out:=pointcloud</argument>
+            </ros>
+            <!-- Set output to sensor_msgs/PointCloud to get same output type as gazebo_ros_block_laser -->
+            <output_type>sensor_msgs/PointCloud</output_type>
+            <!-- <frame_name> ommited, will default to block_laser_link -->
+            <!-- min_intensity instead of hokuyoMinIntensity -->
+            <min_intensity>100.0</min_intensity>
+            </plugin>
+        </sensor>
+    </gazebo>
+</xacro:macro>
 </robot>

Commit message: Added solutions for pc and world models

File: box_bot_description/robot/box_bot_with_meshes.xacro (robot description, xacro)
@@ -17,5 +17,5 @@
   <xacro:caster_wheel parent="chassis" caster_wheel_name="back" origin_xyz="${(-1.0 *base_box_x / 2.0) + wheel_increment} 0 ${-1.0* base_box_x / 2.0}" radius="${wheel_increment}" legth="${dummy_length}"/>
   <xacro:camera_rgb parent_name="${base_name}" sensor_name="rgb_camera" origin_xyz="${base_box_x/ 1.9} 0.0 ${base_box_x / 2.0}" camera_ROLL="0.0" camera_PITCH="0.0" camera_YAW="0.0"/>
-  <xacro:laser_scan parent_name="${base_name}" sensor_name="laser_scan" origin_xyz="0.0 0.0 ${base_box_x / 1.5}" sensor_YAW="1.57"/>
+  <xacro:laser_scan parent_name="${base_name}" sensor_name="laser_scan" origin_xyz="0.0 0.0 ${base_box_x / 2.0}" sensor_YAW="1.57"/>
   <xacro:block_laser_scan parent_name="${base_name}" sensor_name="block_laser_scan" origin_xyz="${base_box_x/ 1.9} 0.0 ${base_box_x / 2.0}" sensor_YAW="1.57"/>
 </robot>

File: box_bot_description/robot/sensors.xacro (robot description, xacro)
@@ -32,11 +32,11 @@
                 <horizontal_fov>1.3962634</horizontal_fov>
                 <image>
-                <width>800</width>
-                <height>800</height>
+                <width>300</width>
+                <height>300</height>
                 <format>R8G8B8</format>
                 </image>
                 <clip>
                 <near>0.02</near>
-                <far>300</far>
+                <far>20.0</far>
                 </clip>
                 <noise>
@@ -48,4 +48,6 @@
                 <stddev>0.007</stddev>
                 </noise>
+                <always_on>1</always_on>
+                <update_rate>30</update_rate>
             </camera>
             <plugin name="plugin_name" filename="libgazebo_ros_camera.so">
@@ -150,5 +152,5 @@
     </link>
     <joint name="${sensor_name}_laser_scan_frame_joint" type="fixed">
-        <origin xyz="0 0 0" rpy="0 0 0" />
+        <origin xyz="0 0 0.03" rpy="0 0 0" />
         <parent link="${sensor_name}_laser_scan_link" />
         <child link="${sensor_name}_laser_scan_frame" />
@@ -157,5 +159,5 @@
 	<gazebo reference="${sensor_name}_laser_scan_frame">
 		<sensor name="sensor_ray" type="ray">
-        <pose>0.5 0 0 0 0 0</pose>
+        <pose>0 0 0 0 0 0</pose>
         <ray>
           <scan>
