Commit message: Added working sensor clean two robot launch

File: box_bot_description/robot/box_bot_laser_control.xacro (robot description, xacro)
@@ -1,5 +1,5 @@
 <?xml version="1.0"?>
 <robot xmlns:xacro="http://www.ros.org/wiki/xacro">
-    <xacro:macro  name="box_bot_laser_control" params="robot_name parent">
+    <xacro:macro  name="box_bot_custom_control" params="robot_name parent">
       <link name="${robot_name}_laser_scan_link">
         <visual name="${robot_name}_visual_laser_scan_link">
@@ -57,6 +57,5 @@
         <dynamics friction="0.01"/>
       </joint>
-      <!-- Position Config -->
-        <ros2_control name="GazeboSystem" type="system">
+      <ros2_control name="${robot_name}_GazeboSystem" type="system">
           <hardware>
             <plugin>gazebo_ros2_control/GazeboSystem</plugin>
@@ -82,7 +81,7 @@
       </ros2_control>
       <gazebo>
-        <plugin filename="libgazebo_ros2_control.so" name="gazebo_ros2_control">
+        <plugin filename="libgazebo_ros2_control.so" name="${robot_name}_gazebo_ros2_control">
           <ros>
-            <namespace>/${robot_name}</namespace>
+            <namespace>${robot_name}</namespace>
           </ros>
           <parameters>$(find box_bot_description)/config/${robot_name}_controller_position_velocity.yaml</parameters>

File: box_bot_description/robot/box_bot_with_control.xacro (robot description, xacro)
@@ -8,5 +8,8 @@
   <xacro:include filename="$(find box_bot_description)/robot/box_bot_body.xacro" />
   <xacro:include filename="$(find box_bot_description)/robot/sensors.xacro" />
+  <!-- THIS ORDER IS CRITICAL -->
+  <xacro:include filename="$(find box_bot_description)/robot/box_bot_laser_control.xacro" />
   <xacro:include filename="$(find box_bot_description)/robot/box_bot.gazebo" />
+  <!-- END -->
   <xacro:arg name="box_bot_name" default="box_bot"/>
   <xacro:box_bot_body robot_name="$(arg box_bot_name)"/>
@@ -15,7 +18,7 @@
   <xacro:caster_wheel robot_name="$(arg box_bot_name)" parent="$(arg box_bot_name)_chassis" caster_wheel_name="front" origin_xyz="${(base_box_x / 2.0) - wheel_increment} 0 ${-1.0* base_box_x / 2.0}" radius="${wheel_increment}" legth="${dummy_length}"/>
   <xacro:caster_wheel robot_name="$(arg box_bot_name)" parent="$(arg box_bot_name)_chassis" caster_wheel_name="back" origin_xyz="${(-1.0 *base_box_x / 2.0) + wheel_increment} 0 ${-1.0* base_box_x / 2.0}" radius="${wheel_increment}" legth="${dummy_length}"/>
+  <xacro:box_bot_custom_control robot_name="$(arg box_bot_name)" parent="$(arg box_bot_name)_chassis"/>
   <xacro:box_bot_gazebo_systems robot_name="$(arg box_bot_name)"/>
-  <xacro:laser_scan robot_name="$(arg box_bot_name)" parent_name="$(arg box_bot_name)_chassis" origin_xyz="0.0 0.0 ${base_box_x / 2.0}" sensor_YAW="0.0"/>
-  <xacro:point_cloud_sensor robot_name="$(arg box_bot_name)" parent_name="$(arg box_bot_name)_chassis" sensor_name="block_laser_scan" origin_xyz="${base_box_x/ 1.9} 0.0 0.0" sensor_YAW="0.0"/>
+  <xacro:laser_scan robot_name="$(arg box_bot_name)" parent_name="$(arg box_bot_name)_laser_scan_link" origin_xyz="0.0 0.0 ${base_box_x / 2.0}" sensor_YAW="0.0"/>
   <xacro:camera_rgb robot_name="$(arg box_bot_name)" parent_name="$(arg box_bot_name)_chassis" origin_xyz="${base_box_x/ 1.9} 0.0 ${base_box_x / 2.0}" camera_ROLL="0.0" camera_PITCH="0.0" camera_YAW="0.0"/>
 </robot>

File: box_bot_description/robot/sensors_for_control.xacro (robot description, xacro)
@@ -39,5 +39,4 @@
           <plugin name="camera_controller" filename="libgazebo_ros_camera.so">
             <ros>
-              <namespace>${robot_name}</namespace>
             </ros>
             <cameraName>${robot_name}_rgb_camera</cameraName>
@@ -51,33 +50,9 @@
   </xacro:macro>
   <xacro:macro name="laser_scan" params="robot_name parent_name origin_xyz sensor_YAW">
-      <link name="${robot_name}_laser_scan_model_link">
-        <visual name="${robot_name}_visual_laser_scan_link">
-          <origin rpy="0 0 0" xyz="0 0 0"/>
-          <geometry>
-            <mesh filename="package://box_bot_description/meshes/sensors/rplidar.dae" scale="1.0 1.0 1.0"/>
-          </geometry>
-        </visual>
-        <collision name="${robot_name}_collision_laser_scan_link">
-          <origin rpy="0 0 0" xyz="0 0 0.0204"/>
-          <geometry>
-            <cylinder length="0.0408" radius="0.037493"/>
-          </geometry>
-        </collision>
-        <inertial>
-          <mass value="0.01"/>
-          <origin rpy="0 0 0" xyz="0 0 0.0204"/>
-          <inertia ixx="6.066578520833334e-06" ixy="0" ixz="0" iyy="6.066578520833334e-06" iyz="0" izz="9.365128684166666e-06"/>
-        </inertial>
-      </link>
-    <joint name="${robot_name}_laser_scan_model_link_joint" type="fixed">
-        <origin xyz="${origin_xyz}" rpy="0 0 ${sensor_YAW}" />
-        <parent link="${parent_name}" />
-        <child link="${robot_name}_laser_scan_model_link" />
-    </joint>
     <link name="${robot_name}_laser_scan_frame">
     </link>
     <joint name="${robot_name}_laser_scan_frame_joint" type="fixed">
-        <origin xyz="0 0 0.03" rpy="0 0 ${sensor_YAW}" />
-        <parent link="${robot_name}_laser_scan_model_link" />
+        <origin xyz="${origin_xyz}" rpy="0 0 ${sensor_YAW}" />
+        <parent link="${parent_name}" />
         <child link="${robot_name}_laser_scan_frame" />
     </joint>
@@ -104,6 +79,5 @@
           <plugin name="laser" filename="libgazebo_ros_ray_sensor.so">
             <ros>
-              <namespace>${robot_name}</namespace>
-              <remapping>~/out:=laser_scan</remapping>
+              <remapping>~/out:=${robot_name}/laser_scan</remapping>
             </ros>
             <output_type>sensor_msgs/LaserScan</output_type>
@@ -154,6 +128,5 @@
             <!-- Change namespace and output topic so published topic is /rrbot/laser/pointcloud -->
             <ros>
-                <namespace>${robot_name}</namespace>
-                <argument>--ros-args --remap ~/out:=pointcloud</argument>
+                <argument>--ros-args --remap ~/out:=${robot_name}/pointcloud</argument>
             </ros>
             <!-- Set output to sensor_msgs/PointCloud to get same output type as gazebo_ros_block_laser -->
