Commit message: Added corrections

File: box_bot_description/robot/wheels.xacro (robot description, xacro)
@@ -27,5 +27,5 @@
         <mu1>${mu1_wheel}</mu1>
         <mu2>${mu2_wheel}</mu2>
-        <material>Gazebo/Blue</material>
+        <material>Gazebo/White</material>
       </gazebo>
   </xacro:macro >

Commit message: Added mods for slotcar

File: box_bot_description/robot/wheels.xacro (robot description, xacro)
@@ -29,7 +29,7 @@
         <material>Gazebo/White</material>
       </gazebo>
-      <joint name="${robot_name}_${name_wheel_link}_joint" type="continuous">
+      <joint name="${robot_name}/joint_tire_${name_wheel_link}" type="continuous">
         <origin rpy="0 0 0" xyz="${origin_xyz}"/>
-        <child link="${child}"/>
+        <child link="${robot_name}_${name_wheel_link}"/>
         <parent link="${parent}"/>
         <axis rpy="0 0 0" xyz="0 1 0"/>
