Commit message: Added try for colours fix in melodic without any luck

File: box_bot_description/robot/box_bot_body.xacro (robot description, xacro)
@@ -12,14 +12,13 @@
         </inertial>
         <!-- body -->
-        <collision name="collision_chassis">
+        <collision name="collision_${parent_name}">
           <geometry>
             <box size="${base_box_x} ${base_box_y} ${base_box_z}"/>
           </geometry>
         </collision>
-        <visual name="visual_chassis">
+        <visual name="visual_${parent_name}">
           <geometry>
             <box size="${base_box_x} ${base_box_y} ${base_box_z}"/>
           </geometry>
-          <material name="red"/>
         </visual>
       </link>

Commit message: Added corrections

File: box_bot_description/robot/box_bot_body.xacro (robot description, xacro)
@@ -34,3 +34,40 @@
       </joint>
     </xacro:macro >
+    <!-- box_bot_body_with_meshes -->
+    <xacro:macro  name="box_bot_body_with_meshes" params="parent_name">
+      <link name="base_link">
+      </link>
+      <link name="${parent_name}">
+        <!-- pose and inertial -->
+        <pose>0 0 0 0 0 0</pose>
+        <inertial>
+          <mass value="${base_box_mass}"/>
+          <origin rpy="0 0 0" xyz="0 0 0"/>
+          <xacro:box_inertia mass="0.2" x="${base_box_x}" y="${base_box_y}" z="${base_box_z}"/>
+          <inertia ixx="0.000241935" ixy="0" ixz="0" iyy="0.000241935" iyz="0" izz="0.000241935"/>
+        </inertial>
+        <!-- body -->
+        <collision name="collision_${parent_name}">
+          <geometry>
+                <mesh filename="$(find box_bot_description)/meshes/cute_cube.dae" scale="${base_box_x} ${base_box_y} ${base_box_z}"/>
+          </geometry>
+        </collision>
+        <visual name="visual_${parent_name}">
+          <geometry>
+                <mesh filename="$(find box_bot_description)/meshes/cute_cube.dae" scale="${base_box_x} ${base_box_y} ${base_box_z}"/>
+          </geometry>
+        </visual>
+        <animation name="animation">
+          <filename>Idle.dae</filename>
+        </animation>
+      </link>
+      <gazebo reference="${parent_name}">
+        <material>Gazebo/Red</material>
+      </gazebo>
+      <joint name="base_link_joint" type="fixed">
+        <origin rpy="0 0 0" xyz="0 0 0" />
+        <parent link="base_link" />
+        <child link="${parent_name}" />
+      </joint>
+    </xacro:macro >
 </robot>

File: box_bot_description/robot/wheels.xacro (robot description, xacro)
@@ -9,5 +9,5 @@
               <xacro:cylinder_inertia mass="0.2" r="${r}" l="${l}" />
           </inertial>
-          <collision name="link_right_wheel_collision">
+          <collision name="${name}_collision">
             <origin rpy="0 1.5707 1.5707" xyz="0 0 0"/>
             <geometry>
@@ -15,5 +15,5 @@
             </geometry>
           </collision>
-          <visual name="link_right_wheel_visual">
+          <visual name="${name}_visual">
             <origin rpy="0 1.5707 1.5707" xyz="0 0 0"/>
             <geometry>
@@ -22,4 +22,11 @@
           </visual>
       </link>
+      <gazebo reference="${name}">
+        <kp>${kp_wheel}</kp>
+        <kd>${kd_wheel}</kd>
+        <mu1>${mu1_wheel}</mu1>
+        <mu2>${mu2_wheel}</mu2>
+        <material>Gazebo/Blue</material>
+      </gazebo>
   </xacro:macro >
   <xacro:macro  name="joint_wheel" params="name parent child origin_xyz">

Commit message: Adding working sensors and tfs

File: box_bot_description/robot/box_bot_body.xacro (robot description, xacro)
@@ -2,6 +2,4 @@
 <robot xmlns:xacro="http://www.ros.org/wiki/xacro">
     <xacro:macro  name="box_bot_body" params="parent_name">
-      <link name="base_link">
-      </link>
       <link name="${parent_name}">
         <!-- pose and inertial -->
@@ -28,14 +26,7 @@
         <material>Gazebo/Red</material>
       </gazebo>
-      <joint name="base_link_joint" type="fixed">
-        <origin rpy="0 0 0" xyz="0 0 0" />
-        <parent link="base_link" />
-        <child link="${parent_name}" />
-      </joint>
     </xacro:macro >
     <!-- box_bot_body_with_meshes -->
     <xacro:macro  name="box_bot_body_with_meshes" params="parent_name">
-      <link name="base_link">
-      </link>
       <link name="${parent_name}">
         <!-- pose and inertial -->
@@ -65,9 +56,4 @@
         <material>Gazebo/Red</material>
       </gazebo>
-      <joint name="base_link_joint" type="fixed">
-        <origin rpy="0 0 0" xyz="0 0 0" />
-        <parent link="base_link" />
-        <child link="${parent_name}" />
-      </joint>
     </xacro:macro >
 </robot>

File: box_bot_description/robot/box_bot_with_meshes.xacro (robot description, xacro)
@@ -8,4 +8,5 @@
   <xacro:include filename="$(find box_bot_description)/robot/box_bot_body.xacro" />
   <xacro:include filename="$(find box_bot_description)/robot/box_bot.gazebo" />
+  <xacro:include filename="$(find box_bot_description)/robot/sensors.xacro" />
   <xacro:box_bot_body_with_meshes parent_name="${base_name}"/>
   <xacro:link_wheel name="right_wheel" r="${wheel_radius}" l="${wheel_width}" incr="${wheel_increment}"/>
@@ -15,3 +16,5 @@
   <xacro:caster_wheel parent="chassis" caster_wheel_name="front" origin_xyz="${(base_box_x / 2.0) - wheel_increment} 0 ${-1.0* base_box_x / 2.0}" radius="${wheel_increment}" legth="${dummy_length}"/>
   <xacro:caster_wheel parent="chassis" caster_wheel_name="back" origin_xyz="${(-1.0 *base_box_x / 2.0) + wheel_increment} 0 ${-1.0* base_box_x / 2.0}" radius="${wheel_increment}" legth="${dummy_length}"/>
+  <!-- <xacro:camera_rgb parent_name="${base_name}" sensor_name="rgb_camera" origin_xyz="${base_box_x} 0.0 ${base_box_x / 2.0}" camera_ROLL="0.0" camera_PITCH="0.0" camera_YAW="0.0"/>
+  <xacro:laser_scan parent_name="${base_name}" sensor_name="rgb_camera" origin_xyz="${base_box_x} 0.0 ${base_box_x / 2.0}" sensor_YAW="0.0"/> -->
 </robot>

File: box_bot_description/robot/properties.xacro (robot description, xacro)
@@ -19,3 +19,19 @@
     <!--Caster Wheels-->
     <xacro:property name="dummy_length" value="0.001"/>
+    <!-- Sensors -->
+    <xacro:property name="sensor_mass" value="0.01"/>
+    <xacro:property name="camera_box_x" value="0.02"/>
+    <xacro:property name="camera_box_y" value="0.01"/>
+    <xacro:property name="camera_box_z" value="0.01"/>
+    <!-- Oberc Astra-->
+    <xacro:property name="orbbec_astra_scale" value="1.0"/>
+    <!-- RGB sensor - cam -->
+    <xacro:property name="orbbec_astra_rel_rgb_px"   value="0.0" />
+    <xacro:property name="orbbec_astra_rel_rgb_py"   value="-0.0125" />
+    <xacro:property name="orbbec_astra_rel_rgb_pz"   value="-0.0150" />
+    <!-- IR sensor - depth -->
+    <xacro:property name="orbbec_astra_depth_rel_rgb_px" value="0.0" />
+    <xacro:property name="orbbec_astra_depth_rel_rgb_py" value="0.0250" />
+    <xacro:property name="orbbec_astra_depth_rel_rgb_pz" value="0.0" />
+    <xacro:property name="M_PI" value="3.1415926535897931" />
 </robot>

Commit message: Added and solved issue with tfs and meshes added small rplydar model

File: box_bot_description/robot/box_bot_body.xacro (robot description, xacro)
@@ -41,10 +41,12 @@
         <collision name="collision_${parent_name}">
           <geometry>
-                <mesh filename="$(find box_bot_description)/meshes/cute_cube.dae" scale="${base_box_x} ${base_box_y} ${base_box_z}"/>
+                <!-- <mesh filename="$(find box_bot_description)/meshes/cute_cube.dae" scale="${base_box_x} ${base_box_y} ${base_box_z}"/> -->
+                <mesh filename="package://box_bot_description/meshes/cute_cube.dae" scale="${base_box_x} ${base_box_y} ${base_box_z}"/>
           </geometry>
         </collision>
         <visual name="visual_${parent_name}">
           <geometry>
-                <mesh filename="$(find box_bot_description)/meshes/cute_cube.dae" scale="${base_box_x} ${base_box_y} ${base_box_z}"/>
+                <!-- <mesh filename="$(find box_bot_description)/meshes/cute_cube.dae" scale="${base_box_x} ${base_box_y} ${base_box_z}"/> -->
+                <mesh filename="package://box_bot_description/meshes/cute_cube.dae" scale="${base_box_x} ${base_box_y} ${base_box_z}"/>
           </geometry>
         </visual>

File: box_bot_description/robot/box_bot_with_meshes.xacro (robot description, xacro)
@@ -16,5 +16,5 @@
   <xacro:caster_wheel parent="chassis" caster_wheel_name="front" origin_xyz="${(base_box_x / 2.0) - wheel_increment} 0 ${-1.0* base_box_x / 2.0}" radius="${wheel_increment}" legth="${dummy_length}"/>
   <xacro:caster_wheel parent="chassis" caster_wheel_name="back" origin_xyz="${(-1.0 *base_box_x / 2.0) + wheel_increment} 0 ${-1.0* base_box_x / 2.0}" radius="${wheel_increment}" legth="${dummy_length}"/>
-  <!-- <xacro:camera_rgb parent_name="${base_name}" sensor_name="rgb_camera" origin_xyz="${base_box_x} 0.0 ${base_box_x / 2.0}" camera_ROLL="0.0" camera_PITCH="0.0" camera_YAW="0.0"/>
-  <xacro:laser_scan parent_name="${base_name}" sensor_name="rgb_camera" origin_xyz="${base_box_x} 0.0 ${base_box_x / 2.0}" sensor_YAW="0.0"/> -->
+  <xacro:camera_rgb parent_name="${base_name}" sensor_name="rgb_camera" origin_xyz="${base_box_x} 0.0 ${base_box_x / 2.0}" camera_ROLL="0.0" camera_PITCH="0.0" camera_YAW="0.0"/>
+  <xacro:laser_scan parent_name="${base_name}" sensor_name="laser_scan" origin_xyz="0.0 0.0 ${base_box_x / 2.0}" sensor_YAW="0.0"/>
 </robot>

File: box_bot_description/robot/sensors.xacro (robot description, xacro)
@@ -135,4 +135,9 @@
   <xacro:macro name="laser_scan" params="parent_name sensor_name origin_xyz sensor_YAW">
     <link name='${sensor_name}_laser_scan_link'>
+        <visual name="visual_${parent_name}">
+            <geometry>
+                    <mesh filename="package://box_bot_description/meshes/sensors/rplidar.dae" scale="${base_box_x} ${base_box_y} ${base_box_z}"/>
+            </geometry>
+        </visual>
 	</link>
     <joint name="${sensor_name}_laser_scan_link_joint" type="fixed">

Commit message: Added three colour versions

File: box_bot_description/robot/box_bot_body.xacro (robot description, xacro)
@@ -7,5 +7,5 @@
         <visual name="${robot_name}_visual_chassis">
           <geometry>
-            <mesh filename="package://box_bot_description/meshes/cute_cube.dae" scale="0.1 0.1 0.1"/>
+            <mesh filename="package://box_bot_description/meshes/${robot_name}.dae" scale="0.1 0.1 0.1"/>
           </geometry>
           <material name="box_bot_blue"/>

File: box_bot_description/robot/sensors.xacro (robot description, xacro)
@@ -100,5 +100,5 @@
           </ray>
           <always_on>true</always_on>
-          <visualize>true</visualize>
+          <visualize>false</visualize>
           <update_rate>100.0</update_rate>
           <plugin name="laser" filename="libgazebo_ros_ray_sensor.so">

Commit message: Added mods to make rmf slotcar work

File: box_bot_description/robot/box_bot_body.xacro (robot description, xacro)
@@ -5,11 +5,10 @@
       </link>
       <link name="${robot_name}_chassis">
-        <visual name="${robot_name}_visual_chassis">
+        <visual>
           <geometry>
-            <mesh filename="package://box_bot_description/meshes/${robot_name}.dae" scale="0.1 0.1 0.1"/>
+            <mesh filename="package://box_bot_description/meshes/box_bot_1.dae" scale="0.1 0.1 0.1"/>
           </geometry>
-          <material name="box_bot_blue"/>
         </visual>
-        <collision name="${robot_name}_collision_chassis">
+        <collision>
           <geometry>
             <box size="0.1 0.1 0.1"/>

File: box_bot_description/robot/box_bot_slotcar.xacro (robot description, xacro)
@@ -9,8 +9,8 @@
   <xacro:include filename="$(find box_bot_description)/robot/sensors.xacro" />
   <xacro:include filename="$(find box_bot_description)/robot/box_bot.gazebo" />
-  <xacro:arg name="box_bot_name" default="box_bot"/>
+  <xacro:arg name="box_bot_name" default="box_bot_1"/>
   <xacro:box_bot_body robot_name="$(arg box_bot_name)"/>
-  <xacro:wheel parent="$(arg box_bot_name)_chassis" child="$(arg box_bot_name)_right_wheel" origin_xyz="0 ${base_box_x / 2.0} ${-1.0 * wheel_radius}" robot_name="$(arg box_bot_name)" name_wheel_link="right" r="${wheel_radius}" l="${wheel_width}" incr="${wheel_increment}"/>
-  <xacro:wheel parent="$(arg box_bot_name)_chassis" child="$(arg box_bot_name)_left_wheel" origin_xyz="0 ${-1.0 * base_box_x / 2.0} ${-1.0 * wheel_radius}" robot_name="$(arg box_bot_name)" name_wheel_link="left" r="${wheel_radius}" l="${wheel_width}" incr="${wheel_increment}"/>
+  <xacro:wheel parent="$(arg box_bot_name)_chassis" child="$(arg box_bot_name)_left_wheel" origin_xyz="0 ${base_box_x / 2.0} ${-1.0 * wheel_radius}" robot_name="$(arg box_bot_name)" name_wheel_link="left" r="${wheel_radius}" l="${wheel_width}" incr="${wheel_increment}"/>
+  <xacro:wheel parent="$(arg box_bot_name)_chassis" child="$(arg box_bot_name)_right_wheel" origin_xyz="0 ${-1.0 * base_box_x / 2.0} ${-1.0 * wheel_radius}" robot_name="$(arg box_bot_name)" name_wheel_link="right" r="${wheel_radius}" l="${wheel_width}" incr="${wheel_increment}"/>
   <xacro:caster_wheel robot_name="$(arg box_bot_name)" parent="$(arg box_bot_name)_chassis" caster_wheel_name="front" origin_xyz="${(base_box_x / 2.0) - wheel_increment} 0 ${-1.0* base_box_x / 2.0}" radius="${wheel_increment}" legth="${dummy_length}"/>
   <xacro:caster_wheel robot_name="$(arg box_bot_name)" parent="$(arg box_bot_name)_chassis" caster_wheel_name="back" origin_xyz="${(-1.0 *base_box_x / 2.0) + wheel_increment} 0 ${-1.0* base_box_x / 2.0}" radius="${wheel_increment}" legth="${dummy_length}"/>
