Commit message: Adding working boxbot

File: box_bot_description/robot/box_bot.xacro (robot description, xacro)
@@ -1,12 +1,22 @@
 <?xml version="1.0" ?>
 <robot name="box_bot" xmlns:xacro="http://www.ros.org/wiki/xacro">
-  <xacro:include filename="$(find box_bot_description)/urdf/materials.xacro" />
-  <xacro:include filename="$(find box_bot_description)/urdf/box_bot.gazebo" />
-  <xacro:include filename="$(find box_bot_description)/urdf/macros.xacro" />
-  <xacro:include filename="$(find box_bot_description)/urdf/box_bot_body.xacro" />
-  <xacro:link_wheel name="link_right_wheel" r="0.0381" l="0.001" incr="0.002"/>
-  <xacro:joint_wheel name="joint_right_wheel" child="link_right_wheel" origin_xyz="0 0.0181 0" />
-  <xacro:link_wheel name="link_left_wheel" r="0.0381" l="0.001" incr="0.002"/>
-  <xacro:joint_wheel name="joint_left_wheel" child="link_left_wheel" origin_xyz="0 -0.0181 0" />
-  <xacro:box_bot_dummy  name="box_bot_dummy" parent="link_chassis" r="0.0381" l="0.001" incr="0.002"/>
+  <xacro:include filename="$(find box_bot_description)/robot/materials.xacro" />
+  <xacro:include filename="$(find box_bot_description)/robot/properties.xacro" />
+  <xacro:include filename="$(find box_bot_description)/robot/macros.xacro" />
+  <xacro:include filename="$(find box_bot_description)/robot/wheels.xacro" />
+  <xacro:include filename="$(find box_bot_description)/robot/caster_wheels.xacro" />
+  <xacro:include filename="$(find box_bot_description)/robot/box_bot.gazebo" />
+  <xacro:include filename="$(find box_bot_description)/robot/box_bot_body.xacro" />
+  <!--
+  <xacro:include filename="$(find box_bot_description)/robot/box_bot_propeller.xacro" />
+  -->
+  <xacro:box_bot_body parent_name="chassis"/>
+  <!--
+  <xacro:link_wheel name="link_right_wheel" r="${wheel_radius}" l="${wheel_width}" incr="${wheel_increment}"/>
+  <xacro:joint_wheel name="joint_right_wheel" child="link_right_wheel" origin_xyz="0 ${base_box_x / 4.0} 0" />
+  <xacro:link_wheel name="link_left_wheel" r="${wheel_radius}" l="${wheel_width}" incr="${wheel_increment}"/>
+  <xacro:joint_wheel name="joint_left_wheel" child="link_left_wheel" origin_xyz="0 ${-1.0 * base_box_x / 2.0} 0" />
+  <xacro:caster_wheel parent="chassis" caster_wheel_name="front" origin_xyz="${base_box_x / 2.0} 0 0" />
+  <xacro:caster_wheel parent="chassis" caster_wheel_name="front" origin_xyz="${-1.0 *base_box_x / 2.0} 0 0" />
+  -->
 </robot>

File: box_bot_description/robot/box_bot_body.xacro (robot description, xacro)
@@ -1,20 +1,12 @@
 <?xml version="1.0"?>
 <robot xmlns:xacro="http://www.ros.org/wiki/xacro">
-    <xacro:macro  name="box_bot_body" params="name parent l r incr">
-      <!-- ros_control plugin -->
-        <gazebo>
-          <plugin name="gazebo_ros_control"
-                  filename="libgazebo_ros_control.so">
-            <robotNamespace>/box_bot</robotNamespace>
-            <robotParam>/robot_description</robotParam>
-            <robotSimType>gazebo_ros_control/DefaultRobotHWSim</robotSimType>
-          </plugin>
-        </gazebo>
-      <link name="${parent}">
+    <xacro:macro  name="box_bot_body" params="parent_name">
+      <link name="${parent_name}">
         <!-- pose and inertial -->
         <pose>0 0 0 0 0 0</pose>
         <inertial>
-          <mass value="1"/>
+          <mass value="${base_box_mass}"/>
           <origin rpy="0 0 0" xyz="0 0 0"/>
+          <box_inertia mass="0.2" x="${base_box_x}" y="${base_box_y}" z="${base_box_z}"/>
           <inertia ixx="0.000241935" ixy="0" ixz="0" iyy="0.000241935" iyz="0" izz="0.000241935"/>
         </inertial>
@@ -22,44 +14,13 @@
         <collision name="collision_chassis">
           <geometry>
-            <box size="0.0762 0.0762 0.0762"/>
+            <box size="${base_box_x} ${base_box_y} ${base_box_z}"/>
           </geometry>
         </collision>
-      </link>
-      <link name="${name}_base_direction_link">
-        <inertial>
-          <mass value="0.2"/>
-          <origin rpy="0 1.5707 1.5707" xyz="0 0 0"/>
-            <cylinder_inertia mass="0.2" r="${r}" l="${l}" />
-        </inertial>
-        <collision name="link_right_wheel_collision">
-          <origin rpy="0 1.5707 1.5707" xyz="0 0 0"/>
+        <visual name="visual_chassis">
           <geometry>
-            <cylinder length="${l}" radius="${r + incr}"/>
-          </geometry>
-        </collision>
-        <visual>
-          <origin rpy="0 0 0" xyz="0 0.0 0.0" />
-          <geometry>
-            <mesh filename="package://box_bot_description/meshes/box_bot_Textured.dae" scale="1.3 1.3 1.3"/>
+            <box size="${base_box_x} ${base_box_y} ${base_box_z}"/>
           </geometry>
         </visual>
       </link>
-      <joint name="direction_joint" type="continuous">
-        <origin rpy="0 0 0" xyz="0.0 0.0 0.0" />
-        <parent link="${parent}" />
-        <child link="${name}_base_direction_link" />
-        <axis xyz="0 1 0" />
-        <limit effort="1000.0" velocity="100.0" />
-      </joint>
-    <transmission name="direction_joint_trans">
-      <type>transmission_interface/SimpleTransmission</type>
-      <joint name="direction_joint">
-        <hardwareInterface>EffortJointInterface</hardwareInterface>
-      </joint>
-      <actuator name="direction_jointMotor">
-        <hardwareInterface>EffortJointInterface</hardwareInterface>
-        <mechanicalReduction>1</mechanicalReduction>
-      </actuator>
-    </transmission>
     </xacro:macro >
 </robot>

File: box_bot_description/robot/macros.xacro (robot description, xacro)
@@ -6,34 +6,16 @@
                 izz="${mass*(r*r)/2}" />
     </xacro:macro >
-    <xacro:macro  name="link_wheel" params="name r l incr">
-        <link name="${name}">
-            <inertial>
-              <mass value="0.2"/>
-              <origin rpy="0 1.5707 1.5707" xyz="0 0 0"/>
-               <cylinder_inertia mass="0.2" r="${r}" l="${l}" />
-            </inertial>
-            <collision name="link_right_wheel_collision">
-              <origin rpy="0 1.5707 1.5707" xyz="0 0 0"/>
-              <geometry>
-                <cylinder length="${l}" radius="${r + incr}"/>
-              </geometry>
-            </collision>
-            <visual name="link_right_wheel_visual">
-              <origin rpy="0 1.5707 1.5707" xyz="0 0 0"/>
-              <geometry>
-                <cylinder length="${l}" radius="${r + incr}"/>
-              </geometry>
-            </visual>
-        </link>
-    </xacro:macro >
-    <xacro:macro  name="joint_wheel" params="name child origin_xyz">
-      <joint name="${name}" type="continuous">
-        <origin rpy="0 0 0" xyz="${origin_xyz}"/>
-        <child link="${child}"/>
-        <parent link="link_chassis"/>
-        <axis rpy="0 0 0" xyz="0 1 0"/>
-        <limit effort="10000" velocity="1000"/>
-        <joint_properties damping="1.0" friction="1.0"/>
-      </joint>
-    </xacro:macro >
+    <xacro:macro name="box_inertia" params="mass x y z">
+      <inertia  ixx="${mass*(y*y+z*z)/12}" ixy = "0" ixz = "0"
+                iyy="${mass*(x*x+z*z)/12}" iyz = "0"
+                izz="${mass*(x*x+z*z)/12}"
+      />
+    </xacro:macro>
+  <xacro:macro name="sphere_inertia" params="mass r">
+    <inertia
+          ixx="${2*mass*r*r/5}" ixy = "0" ixz = "0"
+          iyy="${2*mass*r*r/5}" iyz = "0"
+          izz="${2*mass*r*r/5}"
+    />
+  </xacro:macro>
 </robot>

Commit message: Have sim for demo

File: box_bot_description/robot/box_bot.xacro (robot description, xacro)
@@ -11,12 +11,10 @@
   <xacro:include filename="$(find box_bot_description)/robot/box_bot_propeller.xacro" />
   -->
-  <xacro:box_bot_body parent_name="chassis"/>
-  <!--
-  <xacro:link_wheel name="link_right_wheel" r="${wheel_radius}" l="${wheel_width}" incr="${wheel_increment}"/>
-  <xacro:joint_wheel name="joint_right_wheel" child="link_right_wheel" origin_xyz="0 ${base_box_x / 4.0} 0" />
-  <xacro:link_wheel name="link_left_wheel" r="${wheel_radius}" l="${wheel_width}" incr="${wheel_increment}"/>
-  <xacro:joint_wheel name="joint_left_wheel" child="link_left_wheel" origin_xyz="0 ${-1.0 * base_box_x / 2.0} 0" />
-  <xacro:caster_wheel parent="chassis" caster_wheel_name="front" origin_xyz="${base_box_x / 2.0} 0 0" />
-  <xacro:caster_wheel parent="chassis" caster_wheel_name="front" origin_xyz="${-1.0 *base_box_x / 2.0} 0 0" />
-  -->
+  <xacro:box_bot_body parent_name="${base_name}"/>
+  <xacro:link_wheel name="right_wheel" r="${wheel_radius}" l="${wheel_width}" incr="${wheel_increment}"/>
+  <xacro:joint_wheel name="joint_right_wheel" parent="${base_name}" child="right_wheel" origin_xyz="0 ${base_box_x / 2.0} ${-1.0 * wheel_radius}" />
+  <xacro:link_wheel name="left_wheel" r="${wheel_radius}" l="${wheel_width}" incr="${wheel_increment}"/>
+  <xacro:joint_wheel name="joint_left_wheel" parent="${base_name}" child="left_wheel" origin_xyz="0 ${-1.0 * base_box_x / 2.0} ${-1.0 * wheel_radius}" />
+  <xacro:caster_wheel parent="chassis" caster_wheel_name="front" origin_xyz="${(base_box_x / 2.0) - wheel_increment} 0 ${-1.0* base_box_x / 2.0}" radius="${wheel_increment}" legth="${dummy_length}"/>
+  <xacro:caster_wheel parent="chassis" caster_wheel_name="back" origin_xyz="${(-1.0 *base_box_x / 2.0) + wheel_increment} 0 ${-1.0* base_box_x / 2.0}" radius="${wheel_increment}" legth="${dummy_length}"/>
 </robot>

File: box_bot_description/robot/box_bot_body.xacro (robot description, xacro)
@@ -21,4 +21,5 @@
             <box size="${base_box_x} ${base_box_y} ${base_box_z}"/>
           </geometry>
+          <material name="red"/>
         </visual>
       </link>

File: box_bot_description/robot/caster_wheels.xacro (robot description, xacro)
@@ -2,5 +2,5 @@
 <robot xmlns:xacro="http://www.ros.org/wiki/xacro">
     <!-- Caster Wheels-->
-    <xacro:macro  name="caster_wheel" params="parent caster_wheel_name origin_xyz">
+    <xacro:macro  name="caster_wheel" params="parent caster_wheel_name origin_xyz radius legth">
       <!-- CASTER FRONT-->
       <link name="${caster_wheel_name}_yaw_link">
@@ -8,10 +8,10 @@
             <mass value="0.001"/>
             <origin rpy="0 1.5707 1.5707" xyz="0 0 0"/>
-            <cylinder_inertia mass="0.001" r="${r/2.0}" l="${l}" />
+            <cylinder_inertia mass="0.001" r="${0.9 * radius/2.0}" l="${legth}" />
           </inertial>
           <collision name="link_right_wheel_collision">
             <origin rpy="0 1.5707 1.5707" xyz="0 0 0"/>
             <geometry>
-              <cylinder length="${l}" radius="${r/2.0 + incr}"/>
+              <cylinder length="${legth}" radius="${0.9 * radius/2.0}"/>
             </geometry>
           </collision>
@@ -39,10 +39,10 @@
             <mass value="0.001"/>
             <origin rpy="0 1.5707 1.5707" xyz="0 0 0"/>
-            <cylinder_inertia mass="0.001" r="${r/2.0}" l="${l}" />
+            <cylinder_inertia mass="0.001" r="${0.9 * radius/2.0}" l="${legth}" />
           </inertial>
           <collision name="link_right_wheel_collision">
             <origin rpy="0 1.5707 1.5707" xyz="0 0 0"/>
             <geometry>
-              <cylinder length="${l}" radius="${r/2.0 + incr}"/>
+              <cylinder length="${legth}" radius="${0.9 * radius/2.0}"/>
             </geometry>
           </collision>
@@ -70,14 +70,20 @@
           <mass value="0.001"/>
           <origin rpy="0 1.5707 1.5707" xyz="0 0 0"/>
-            <cylinder_inertia mass="0.001" r="${r}" l="${l}" />
+            <sphere_inertia mass="0.001" r="${radius}"/>
         </inertial>
-        <collision name="link_right_wheel_collision">
+        <collision name="${caster_wheel_name}_collision">
           <origin rpy="0 1.5707 1.5707" xyz="0 0 0"/>
           <geometry>
-            <sphere radius="${r + incr}"/>
+            <sphere radius="${radius}"/>
           </geometry>
         </collision>
+        <visual name="${caster_wheel_name}_visual">
+          <origin rpy="0 1.5707 1.5707" xyz="0 0 0"/>
+          <geometry>
+            <sphere radius="${radius}"/>
+          </geometry>
+        </visual>
       </link>
-      <joint name="pitch_joint" type="continuous">
+      <joint name="${caster_wheel_name}_pitch_joint" type="continuous">
         <origin rpy="0 0 0" xyz="0 0 0" />
         <parent link="${caster_wheel_name}_roll_link" />
@@ -97,4 +103,11 @@
       </actuator>
     </transmission>
+    <gazebo reference="${caster_wheel_name}_pitch_link">
+      <kp>1000000000000000000000000000.0</kp>
+      <kd>1000000000000000000000000000.0</kd>
+      <mu1>${mu1_wheel}</mu1>
+      <mu2>${mu2_wheel}</mu2>
+      <material>Gazebo/Green</material>
+    </gazebo>
   </xacro:macro >
 </robot>

File: box_bot_description/robot/properties.xacro (robot description, xacro)
@@ -4,11 +4,18 @@
 	<xacro:property name="PI" value="3.1415926535897931"/>
 	<!-- Base Box -->
+    <xacro:property name="base_name" value="chassis"/>
     <xacro:property name="base_box_mass" value="1.0"/>
-	<xacro:property name="base_box_x" value="0.381"/>
-    <xacro:property name="base_box_y" value="0.381"/>
-    <xacro:property name="base_box_z" value="0.0762"/>
+	<xacro:property name="base_box_x" value="0.1"/>
+    <xacro:property name="base_box_y" value="0.1"/>
+    <xacro:property name="base_box_z" value="0.1"/>
     <!-- Wheels -->
-	<xacro:property name="wheel_radius" value="${base_box_z / 2.0}"/>
+	<xacro:property name="wheel_radius" value="${base_box_z / 4.0}"/>
     <xacro:property name="wheel_width" value="0.001"/>
     <xacro:property name="wheel_increment" value="0.010"/>
+    <xacro:property name="mu1_wheel" value="0.5"/>
+    <xacro:property name="mu2_wheel" value="0.5"/>
+    <xacro:property name="kp_wheel" value="1000.0"/>
+    <xacro:property name="kd_wheel" value="1000.0"/>
+    <!--Caster Wheels-->
+    <xacro:property name="dummy_length" value="0.001"/>
 </robot>

File: box_bot_description/robot/wheels.xacro (robot description, xacro)
@@ -23,9 +23,9 @@
       </link>
   </xacro:macro >
-  <xacro:macro  name="joint_wheel" params="name child origin_xyz">
+  <xacro:macro  name="joint_wheel" params="name parent child origin_xyz">
     <joint name="${name}" type="continuous">
       <origin rpy="0 0 0" xyz="${origin_xyz}"/>
       <child link="${child}"/>
-      <parent link="link_chassis"/>
+      <parent link="${parent}"/>
       <axis rpy="0 0 0" xyz="0 1 0"/>
       <limit effort="10000" velocity="1000"/>

Commit message: No success on fix colour issue

File: box_bot_description/robot/box_bot.xacro (robot description, xacro)
@@ -6,6 +6,6 @@
   <xacro:include filename="$(find box_bot_description)/robot/wheels.xacro" />
   <xacro:include filename="$(find box_bot_description)/robot/caster_wheels.xacro" />
+  <xacro:include filename="$(find box_bot_description)/robot/box_bot_body.xacro" />
   <xacro:include filename="$(find box_bot_description)/robot/box_bot.gazebo" />
-  <xacro:include filename="$(find box_bot_description)/robot/box_bot_body.xacro" />
   <!--
   <xacro:include filename="$(find box_bot_description)/robot/box_bot_propeller.xacro" />

File: box_bot_description/robot/box_bot_body.xacro (robot description, xacro)
@@ -2,4 +2,6 @@
 <robot xmlns:xacro="http://www.ros.org/wiki/xacro">
     <xacro:macro  name="box_bot_body" params="parent_name">
+      <link name="base_link">
+      </link>
       <link name="${parent_name}">
         <!-- pose and inertial -->
@@ -23,4 +25,12 @@
         </visual>
       </link>
+      <gazebo reference="chassis">
+        <material>Gazebo/Red</material>
+      </gazebo>
+      <joint name="base_link_joint" type="fixed">
+        <origin rpy="0 0 0" xyz="0 0 0" />
+        <parent link="base_link" />
+        <child link="${parent_name}" />
+      </joint>
     </xacro:macro >
 </robot>

Commit message: Added camera and laser

File: box_bot_description/robot/box_bot.xacro (robot description, xacro)
@@ -8,4 +8,6 @@
   <xacro:include filename="$(find box_bot_description)/robot/box_bot_body.xacro" />
   <xacro:include filename="$(find box_bot_description)/robot/box_bot.gazebo" />
+  <xacro:arg name="use_nominal_extrinsics" default="false"/>
+  <xacro:include filename="$(find realsense2_description)/urdf/_r430.urdf.xacro" />
   <xacro:box_bot_body parent_name="${base_name}"/>
   <xacro:link_wheel name="right_wheel" r="${wheel_radius}" l="${wheel_width}" incr="${wheel_increment}"/>

File: box_bot_description/robot/box_bot_with_meshes.xacro (robot description, xacro)
@@ -17,4 +17,4 @@
   <xacro:caster_wheel parent="chassis" caster_wheel_name="back" origin_xyz="${(-1.0 *base_box_x / 2.0) + wheel_increment} 0 ${-1.0* base_box_x / 2.0}" radius="${wheel_increment}" legth="${dummy_length}"/>
   <xacro:camera_rgb parent_name="${base_name}" sensor_name="rgb_camera" origin_xyz="${base_box_x} 0.0 ${base_box_x / 2.0}" camera_ROLL="0.0" camera_PITCH="0.0" camera_YAW="0.0"/>
-  <xacro:laser_scan parent_name="${base_name}" sensor_name="laser_scan" origin_xyz="0.0 0.0 ${base_box_x / 2.0}" sensor_YAW="0.0"/>
+  <xacro:laser_scan parent_name="${base_name}" sensor_name="laser_scan" origin_xyz="0.0 0.0 ${base_box_x / 1.5}" sensor_YAW="1.57"/>
 </robot>

File: box_bot_description/robot/sensors.xacro (robot description, xacro)
@@ -184,93 +184,3 @@
 	</gazebo>
   </xacro:macro>
-    <!-- Point Cloud Orbec Astra-->
-  <!-- Xacro properties -->
-  <!--xacro:property name="orbbec_astra_scale" value="0.015"/-->
-  <xacro:macro name="sensor_orbbec_astra" params="prefix parent *origin">
-    <joint name="${prefix}_rgb_joint" type="fixed">
-	  <xacro:insert_block name="origin" />
-      <parent link="${parent}"/>
-      <child link="${prefix}_rgb_base_link" />
-    </joint>
-    <link name="${prefix}_rgb_base_link">
-      <inertial>
-        <mass value="0.001" />
-        <origin xyz="0 0 0" />
-        <inertia ixx="0.0001" ixy="0.0" ixz="0.0"
-          iyy="0.0001" iyz="0.0"
-          izz="0.0001" />
-      </inertial>
-    </link>
-    <joint name="${prefix}_rgb_optical_joint" type="fixed">
-      <origin xyz="0.0 0.0 0.0" rpy="${-M_PI/2} 0 ${-M_PI/2}" />
-      <parent link="${prefix}_rgb_base_link" />
-      <child link="${prefix}_rgb_optical_frame" />
-    </joint>
-    <link name="${prefix}_rgb_optical_frame">
-    </link>
-    <joint name="${prefix}_joint" type="fixed">
-      <origin xyz="${orbbec_astra_rel_rgb_px} ${orbbec_astra_rel_rgb_py} ${orbbec_astra_rel_rgb_pz}"
-              rpy="0.0 0 0"/>
-      <parent link="${prefix}_rgb_base_link"/>
-      <child link="${prefix}_link"/>
-    </joint>
-    <link name="${prefix}_link">
-      <visual>
-        <origin xyz="0 0 ${camera_box_z}" rpy="0 0 0"/>
-        <geometry>
-          <box size="${camera_box_x} ${camera_box_y} ${camera_box_z}"/>
-        </geometry>
-      </visual>
-    </link>
-    <joint name="${prefix}_depth_joint" type="fixed">
-      <origin xyz="${orbbec_astra_depth_rel_rgb_px} ${orbbec_astra_depth_rel_rgb_py} ${orbbec_astra_depth_rel_rgb_pz}" rpy="0 0 0" />
-      <parent link="${prefix}_rgb_base_link" />
-      <child link="${prefix}_depth_frame" />
-    </joint>
-    <link name="${prefix}_depth_frame">
-    </link>
-    <joint name="${prefix}_depth_optical_joint" type="fixed">
-      <origin xyz="0 0 0" rpy="${-M_PI/2} 0 ${-M_PI/2}" />
-      <parent link="${prefix}_depth_frame" />
-      <child link="${prefix}_depth_optical_frame" />
-    </joint>
-    <link name="${prefix}_depth_optical_frame">
-    </link>
-    <gazebo reference="${prefix}_rgb_base_link">
-      <sensor type="depth" name="${prefix}_depth_sensor">
-        <always_on>true</always_on>
-        <update_rate>20.0</update_rate>
-        <camera>
-          <horizontal_fov>${60.0*M_PI/180.0}</horizontal_fov>
-          <image>
-            <format>B8G8R8</format>
-            <width>640</width>
-            <height>480</height>
-          </image>
-          <clip>
-            <near>0.05</near>
-            <far>3.5</far>
-          </clip>
-        </camera>
-        <plugin name="${prefix}_controller" filename="libgazebo_ros_openni_kinect.so">
-          <cameraName>${prefix}</cameraName>
-          <alwaysOn>true</alwaysOn>
-          <updateRate>10</updateRate>
-          <imageTopicName>rgb/image_raw</imageTopicName>
-          <depthImageTopicName>depth/image_raw</depthImageTopicName>
-          <pointCloudTopicName>depth/points</pointCloudTopicName>
-          <cameraInfoTopicName>rgb/camera_info</cameraInfoTopicName>
-          <depthImageCameraInfoTopicName>/${prefix}/depth/camera_info</depthImageCameraInfoTopicName>
-          <frameName>${prefix}_depth_optical_frame</frameName>
-          <baseline>0.1</baseline>
-          <distortion_k1>0.0</distortion_k1>
-          <distortion_k2>0.0</distortion_k2>
-          <distortion_k3>0.0</distortion_k3>
-          <distortion_t1>0.0</distortion_t1>
-          <distortion_t2>0.0</distortion_t2>
-          <pointCloudCutoff>0.4</pointCloudCutoff>
-        </plugin>
-      </sensor>
-    </gazebo>
-  </xacro:macro>
 </robot>
