Commit message: Added XACRO working at 80 percent

File: box_bot_description/robot/box_bot.xacro (robot description, xacro)
@@ -8,10 +8,16 @@
   <xacro:include filename="$(find box_bot_description)/robot/box_bot_body.xacro" />
   <xacro:include filename="$(find box_bot_description)/robot/box_bot.gazebo" />
-  <xacro:box_bot_body parent_name="${base_name}"/>
-  <xacro:link_wheel name="right_wheel" r="${wheel_radius}" l="${wheel_width}" incr="${wheel_increment}"/>
-  <xacro:joint_wheel name="joint_right_wheel" parent="${base_name}" child="right_wheel" origin_xyz="0 ${base_box_x / 2.0} ${-1.0 * wheel_radius}" />
-  <xacro:link_wheel name="left_wheel" r="${wheel_radius}" l="${wheel_width}" incr="${wheel_increment}"/>
-  <xacro:joint_wheel name="joint_left_wheel" parent="${base_name}" child="left_wheel" origin_xyz="0 ${-1.0 * base_box_x / 2.0} ${-1.0 * wheel_radius}" />
-  <xacro:caster_wheel parent="chassis" caster_wheel_name="front" origin_xyz="${(base_box_x / 2.0) - wheel_increment} 0 ${-1.0* base_box_x / 2.0}" radius="${wheel_increment}" legth="${dummy_length}"/>
-  <xacro:caster_wheel parent="chassis" caster_wheel_name="back" origin_xyz="${(-1.0 *base_box_x / 2.0) + wheel_increment} 0 ${-1.0* base_box_x / 2.0}" radius="${wheel_increment}" legth="${dummy_length}"/>
+  <xacro:include filename="$(find box_bot_description)/robot/box_bot_laser_control.xacro" />
+  <xacro:include filename="$(find box_bot_description)/robot/sensors.xacro" />
+  <xacro:arg name="box_bot_name" default="box_bot"/>
+  <xacro:box_bot_body robot_name="$(arg box_bot_name)"/>
+  <xacro:wheel parent="$(arg box_bot_name)_chassis" child="$(arg box_bot_name)_right_wheel" origin_xyz="0 ${base_box_x / 2.0} ${-1.0 * wheel_radius}" robot_name="$(arg box_bot_name)" name_wheel_link="right_wheel" r="${wheel_radius}" l="${wheel_width}" incr="${wheel_increment}"/>
+  <xacro:wheel parent="$(arg box_bot_name)_chassis" child="$(arg box_bot_name)_left_wheel" origin_xyz="0 ${-1.0 * base_box_x / 2.0} ${-1.0 * wheel_radius}" robot_name="$(arg box_bot_name)" name_wheel_link="left_wheel" r="${wheel_radius}" l="${wheel_width}" incr="${wheel_increment}"/>
+  <xacro:caster_wheel robot_name="$(arg box_bot_name)" parent="$(arg box_bot_name)_chassis" caster_wheel_name="front" origin_xyz="${(base_box_x / 2.0) - wheel_increment} 0 ${-1.0* base_box_x / 2.0}" radius="${wheel_increment}" legth="${dummy_length}"/>
+  <xacro:caster_wheel robot_name="$(arg box_bot_name)" parent="$(arg box_bot_name)_chassis" caster_wheel_name="back" origin_xyz="${(-1.0 *base_box_x / 2.0) + wheel_increment} 0 ${-1.0* base_box_x / 2.0}" radius="${wheel_increment}" legth="${dummy_length}"/>
+  <xacro:box_bot_gazebo_systems robot_name="$(arg box_bot_name)"/>
+  <xacro:box_bot_laser_control robot_name="$(arg box_bot_name)" parent="$(arg box_bot_name)_chassis"/>
+  <xacro:laser_scan robot_name="$(arg box_bot_name)" parent_name="$(arg box_bot_name)_laser_scan_link" origin_xyz="0.0 0.0 ${base_box_x / 2.0}" sensor_YAW="0.0"/>
+  <xacro:point_cloud_sensor robot_name="$(arg box_bot_name)" parent_name="$(arg box_bot_name)_chassis" sensor_name="block_laser_scan" origin_xyz="${base_box_x/ 1.9} 0.0 ${base_box_x / 2.0}" sensor_YAW="0.0"/>
+  <xacro:camera_rgb robot_name="$(arg box_bot_name)" parent_name="$(arg box_bot_name)_chassis" origin_xyz="${base_box_x/ 1.9} 0.0 ${base_box_x / 2.0}" camera_ROLL="0.0" camera_PITCH="0.0" camera_YAW="0.0"/>
 </robot>

File: box_bot_description/robot/box_bot_body.xacro (robot description, xacro)
@@ -1,61 +1,30 @@
 <?xml version="1.0"?>
 <robot xmlns:xacro="http://www.ros.org/wiki/xacro">
-    <xacro:macro  name="box_bot_body" params="parent_name">
-      <link name="${parent_name}">
-        <!-- pose and inertial -->
-        <pose>0 0 0 0 0 0</pose>
-        <inertial>
-          <mass value="${base_box_mass}"/>
-          <origin rpy="0 0 0" xyz="0 0 0"/>
-          <xacro:box_inertia mass="0.2" x="${base_box_x}" y="${base_box_y}" z="${base_box_z}"/>
-          <inertia ixx="0.000241935" ixy="0" ixz="0" iyy="0.000241935" iyz="0" izz="0.000241935"/>
-        </inertial>
-        <!-- body -->
-        <collision name="collision_${parent_name}">
+    <xacro:macro  name="box_bot_body" params="robot_name">
+      <link name="${robot_name}_base_link">
+      </link>
+      <link name="${robot_name}_chassis">
+        <visual name="${robot_name}_visual_chassis">
           <geometry>
-            <box size="${base_box_x} ${base_box_y} ${base_box_z}"/>
+            <mesh filename="package://box_bot_description/meshes/cute_cube.dae" scale="0.1 0.1 0.1"/>
+          </geometry>
+          <material name="box_bot_blue"/>
+        </visual>
+        <collision name="${robot_name}_collision_chassis">
+          <geometry>
+            <box size="0.1 0.1 0.1"/>
           </geometry>
         </collision>
-        <visual name="visual_${parent_name}">
-          <geometry>
-            <box size="${base_box_x} ${base_box_y} ${base_box_z}"/>
-          </geometry>
-        </visual>
+        <inertial>
+          <mass value="0.5"/>
+          <origin rpy="0 0 0" xyz="0 0 0"/>
+          <inertia ixx="0.0008333333333333335" ixy="0" ixz="0" iyy="0.0008333333333333335" iyz="0" izz="0.0008333333333333335"/>
+        </inertial>
       </link>
-      <gazebo reference="${parent_name}">
-        <material>Gazebo/Red</material>
-      </gazebo>
-    </xacro:macro >
-    <!-- box_bot_body_with_meshes -->
-    <xacro:macro  name="box_bot_body_with_meshes" params="parent_name">
-      <link name="${parent_name}">
-        <!-- pose and inertial -->
-        <pose>0 0 0 0 0 0</pose>
-        <inertial>
-          <mass value="${base_box_mass}"/>
-          <origin rpy="0 0 0" xyz="0 0 0"/>
-          <xacro:box_inertia mass="0.2" x="${base_box_x}" y="${base_box_y}" z="${base_box_z}"/>
-          <inertia ixx="0.000241935" ixy="0" ixz="0" iyy="0.000241935" iyz="0" izz="0.000241935"/>
-        </inertial>
-        <!-- body -->
-        <collision name="collision_${parent_name}">
-          <geometry>
-                <!-- <mesh filename="$(find box_bot_description)/meshes/cute_cube.dae" scale="${base_box_x} ${base_box_y} ${base_box_z}"/> -->
-                <mesh filename="package://box_bot_description/meshes/cute_cube.dae" scale="${base_box_x} ${base_box_y} ${base_box_z}"/>
-          </geometry>
-        </collision>
-        <visual name="visual_${parent_name}">
-          <geometry>
-                <!-- <mesh filename="$(find box_bot_description)/meshes/cute_cube.dae" scale="${base_box_x} ${base_box_y} ${base_box_z}"/> -->
-                <mesh filename="package://box_bot_description/meshes/cute_cube.dae" scale="${base_box_x} ${base_box_y} ${base_box_z}"/>
-          </geometry>
-        </visual>
-        <animation name="animation">
-          <filename>Idle.dae</filename>
-        </animation>
-      </link>
-      <gazebo reference="${parent_name}">
-        <material>Gazebo/Red</material>
-      </gazebo>
+      <joint name="${robot_name}_base_link_joint" type="fixed">
+        <origin rpy="0 0 0" xyz="0 0 0" />
+        <parent link="${robot_name}_base_link" />
+        <child link="${robot_name}_chassis" />
+      </joint>
     </xacro:macro >
 </robot>

File: box_bot_description/robot/caster_wheels.xacro (robot description, xacro)
@@ -2,7 +2,38 @@
 <robot xmlns:xacro="http://www.ros.org/wiki/xacro">
     <!-- Caster Wheels-->
-    <xacro:macro  name="caster_wheel" params="parent caster_wheel_name origin_xyz radius legth">
+    <xacro:macro  name="caster_wheel" params="robot_name parent caster_wheel_name origin_xyz radius legth">
       <!-- CASTER FRONT-->
-      <link name="${caster_wheel_name}_yaw_link">
+      <link name="${robot_name}_${caster_wheel_name}_yaw_link">
+        <inertial>
+            <mass value="0.001"/>
+            <origin rpy="0 1.5707 1.5707" xyz="0 0 0"/>
+            <xacro:cylinder_inertia mass="0.001" r="${0.9 * radius/2.0}" l="${legth}" />
+          </inertial>
+          <collision name="${robot_name}_${caster_wheel_name}_collision">
+            <origin rpy="0 1.5707 1.5707" xyz="0 0 0"/>
+            <geometry>
+              <cylinder length="${legth}" radius="${0.9 * radius/2.0}"/>
+            </geometry>
+          </collision>
+      </link>
+      <joint name="${robot_name}_${caster_wheel_name}_yaw_joint" type="continuous">
+        <origin rpy="0 0 0" xyz="${origin_xyz}" />
+        <parent link="${parent}" />
+        <child link="${robot_name}_${caster_wheel_name}_yaw_link" />
+        <axis xyz="0 0 1" />
+        <limit effort="1000.0" velocity="100.0" />
+        <dynamics damping="0.0" friction="0.1"/>
+      </joint>
+      <transmission name="${robot_name}_${caster_wheel_name}_yaw_joint_trans">
+      <type>transmission_interface/SimpleTransmission</type>
+      <joint name="${robot_name}_${caster_wheel_name}_yaw_joint">
+        <hardwareInterface>EffortJointInterface</hardwareInterface>
+      </joint>
+      <actuator name="${robot_name}_${caster_wheel_name}_yaw_jointMotor">
+        <hardwareInterface>EffortJointInterface</hardwareInterface>
+        <mechanicalReduction>1</mechanicalReduction>
+      </actuator>
+    </transmission>
+    <link name="${robot_name}_${caster_wheel_name}_roll_link">
         <inertial>
             <mass value="0.001"/>
@@ -17,54 +48,23 @@
           </collision>
       </link>
-      <joint name="${caster_wheel_name}_yaw_joint" type="continuous">
-        <origin rpy="0 0 0" xyz="${origin_xyz}" />
-        <parent link="${parent}" />
-        <child link="${caster_wheel_name}_yaw_link" />
-        <axis xyz="0 0 1" />
+      <joint name="${robot_name}_${caster_wheel_name}_roll_joint" type="continuous">
+        <origin rpy="0 0 0" xyz="0 0 0" />
+        <parent link="${robot_name}_${caster_wheel_name}_yaw_link" />
+        <child link="${robot_name}_${caster_wheel_name}_roll_link" />
+        <axis xyz="1 0 0" />
         <limit effort="1000.0" velocity="100.0" />
         <dynamics damping="0.0" friction="0.1"/>
       </joint>
-      <transmission name="${caster_wheel_name}_yaw_joint_trans">
+      <transmission name="${robot_name}_${caster_wheel_name}_roll_joint_trans">
       <type>transmission_interface/SimpleTransmission</type>
-      <joint name="${caster_wheel_name}_yaw_joint">
+      <joint name="${robot_name}_${caster_wheel_name}_roll_joint">
         <hardwareInterface>EffortJointInterface</hardwareInterface>
       </joint>
-      <actuator name="${caster_wheel_name}_yaw_jointMotor">
+      <actuator name="${robot_name}_${caster_wheel_name}_roll_jointMotor">
         <hardwareInterface>EffortJointInterface</hardwareInterface>
         <mechanicalReduction>1</mechanicalReduction>
       </actuator>
     </transmission>
-    <link name="${caster_wheel_name}_roll_link">
-        <inertial>
-            <mass value="0.001"/>
-            <origin rpy="0 1.5707 1.5707" xyz="0 0 0"/>
-            <xacro:cylinder_inertia mass="0.001" r="${0.9 * radius/2.0}" l="${legth}" />
-          </inertial>
-          <collision name="link_right_wheel_collision">
-            <origin rpy="0 1.5707 1.5707" xyz="0 0 0"/>
-            <geometry>
-              <cylinder length="${legth}" radius="${0.9 * radius/2.0}"/>
-            </geometry>
-          </collision>
-      </link>
-      <joint name="${caster_wheel_name}_roll_joint" type="continuous">
-        <origin rpy="0 0 0" xyz="0 0 0" />
-        <parent link="${caster_wheel_name}_yaw_link" />
-        <child link="${caster_wheel_name}_roll_link" />
-        <axis xyz="1 0 0" />
-        <limit effort="1000.0" velocity="100.0" />
-        <dynamics damping="0.0" friction="0.1"/>
-      </joint>
-      <transmission name="${caster_wheel_name}_roll_joint_trans">
-      <type>transmission_interface/SimpleTransmission</type>
-      <joint name="${caster_wheel_name}_roll_joint">
-        <hardwareInterface>EffortJointInterface</hardwareInterface>
-      </joint>
-      <actuator name="${caster_wheel_name}_roll_jointMotor">
-        <hardwareInterface>EffortJointInterface</hardwareInterface>
-        <mechanicalReduction>1</mechanicalReduction>
-      </actuator>
-    </transmission>
-      <link name="${caster_wheel_name}_pitch_link">
+      <link name="${robot_name}_${caster_wheel_name}_pitch_link">
         <inertial>
           <mass value="0.001"/>
@@ -72,5 +72,5 @@
             <xacro:sphere_inertia mass="0.001" r="${radius}"/>
         </inertial>
-        <collision name="${caster_wheel_name}_collision">
+        <collision name="${robot_name}_${caster_wheel_name}_collision">
           <origin rpy="0 1.5707 1.5707" xyz="0 0 0"/>
           <geometry>
@@ -78,5 +78,5 @@
           </geometry>
         </collision>
-        <visual name="${caster_wheel_name}_visual">
+        <visual name="${robot_name}_${caster_wheel_name}_visual">
           <origin rpy="0 1.5707 1.5707" xyz="0 0 0"/>
           <geometry>
@@ -85,23 +85,23 @@
         </visual>
       </link>
-      <joint name="${caster_wheel_name}_pitch_joint" type="continuous">
+      <joint name="${robot_name}_${caster_wheel_name}_pitch_joint" type="continuous">
         <origin rpy="0 0 0" xyz="0 0 0" />
-        <parent link="${caster_wheel_name}_roll_link" />
-        <child link="${caster_wheel_name}_pitch_link" />
+        <parent link="${robot_name}_${caster_wheel_name}_roll_link" />
+        <child link="${robot_name}_${caster_wheel_name}_pitch_link" />
         <axis xyz="0 1 0" />
         <limit effort="1000.0" velocity="100.0" />
         <dynamics damping="0.0" friction="0.1"/>
       </joint>
-    <transmission name="${caster_wheel_name}_pitch_joint_trans">
+    <transmission name="${robot_name}_${caster_wheel_name}_pitch_joint_trans">
       <type>transmission_interface/SimpleTransmission</type>
-      <joint name="${caster_wheel_name}_pitch_joint">
+      <joint name="${robot_name}_${caster_wheel_name}_pitch_joint">
         <hardwareInterface>EffortJointInterface</hardwareInterface>
       </joint>
-      <actuator name="${caster_wheel_name}_pitch_jointMotor">
+      <actuator name="${robot_name}_${caster_wheel_name}_pitch_jointMotor">
         <hardwareInterface>EffortJointInterface</hardwareInterface>
         <mechanicalReduction>1</mechanicalReduction>
       </actuator>
     </transmission>
-    <gazebo reference="${caster_wheel_name}_pitch_link">
+    <gazebo reference="${robot_name}_${caster_wheel_name}_pitch_link">
       <kp>1000000000000000000000000000.0</kp>
       <kd>1000000000000000000000000000.0</kd>

File: box_bot_description/robot/materials.xacro (robot description, xacro)
@@ -1,27 +1,27 @@
 <?xml version="1.0" ?>
 <robot>
-  <material name="black">
-    <color rgba="0.0 0.0 0.0 1.0"/>
+  <material name="red">
+      <color rgba="1.0 0.0 0.0 1"/>
+  </material>
+  <material name="green_light">
+      <color rgba="0.0 1.0 0.0 1"/>
+  </material>
+  <material name="green_dark">
+    <color rgba="0.0 0.5 0.0 1"/>
   </material>
   <material name="blue">
-    <color rgba="0.203125 0.23828125 0.28515625 1.0"/>
+      <color rgba="0.0 0.0 1.0 1"/>
   </material>
-  <material name="green">
-    <color rgba="0.0 0.8 0.0 1.0"/>
+  <material name="yellow">
+      <color rgba="1.0 1.0 0.0 1"/>
   </material>
-  <material name="grey">
-    <color rgba="0.2 0.2 0.2 1.0"/>
-  </material>
-  <material name="orange">
-    <color rgba="1.0 0.423529411765 0.0392156862745 1.0"/>
-  </material>
-  <material name="brown">
-    <color rgba="0.870588235294 0.811764705882 0.764705882353 1.0"/>
-  </material>
-  <material name="red">
-    <color rgba="0.80078125 0.12890625 0.1328125 1.0"/>
+  <material name="black">
+      <color rgba="0.0 0.0 0.0 1"/>
   </material>
   <material name="white">
-    <color rgba="1.0 1.0 1.0 1.0"/>
+      <color rgba="1.0 1.0 1.0 1"/>
+  </material>
+  <material name="box_bot_blue">
+      <color rgba="0.088656 0.428691 0.491021 1"/>
   </material>
 </robot>

File: box_bot_description/robot/properties.xacro (robot description, xacro)
@@ -17,4 +17,8 @@
     <xacro:property name="kp_wheel" value="1000.0"/>
     <xacro:property name="kd_wheel" value="1000.0"/>
+    <xacro:property name="wheel_separation" value="${base_box_x}"/>
+    <xacro:property name="wheel_diameter" value="${(base_box_z / 2.0) + 2.0 * wheel_increment}"/>
+    <xacro:property name="max_wheel_torque" value="1.0"/>
+    <xacro:property name="max_wheel_acceleration" value="2.0"/>
     <!--Caster Wheels-->
     <xacro:property name="dummy_length" value="0.001"/>
