Commit message: Added XACRO working at 80 percent

File: box_bot_description/robot/sensors.xacro (robot description, xacro)
@@ -1,91 +1,14 @@
 <?xml version="1.0" ?>
 <robot xmlns:xacro="http://www.ros.org/wiki/xacro">
-  <xacro:macro name="camera_rgb" params="parent_name sensor_name origin_xyz camera_ROLL camera_PITCH camera_YAW">
-    <link name='${sensor_name}_camera_link'>
-		<visual>
-			<origin xyz="0 0 0"
-					rpy="0 0 0"/>
-			<geometry>
-				<!-- <box size="${camera_box_x} ${camera_box_y} ${camera_box_z}"/> -->
-                 <mesh filename="package://box_bot_description/meshes/sensors/realsense.dae" scale="0.25 0.25 0.25"/>
-			</geometry>
-		</visual>
-	</link>
-    <joint name="${sensor_name}_camera_link_joint" type="fixed">
-		<origin rpy="${camera_ROLL} ${camera_PITCH} ${camera_YAW}" xyz="${origin_xyz}"/>
-		<parent link="${parent_name}"/>
-		<child link="${sensor_name}_camera_link"/>
-	</joint>
-    <link name="${sensor_name}_camera_link_frame">
+  <xacro:macro name="camera_rgb" params="robot_name parent_name origin_xyz camera_ROLL camera_PITCH camera_YAW">
+    <link name="${robot_name}_rgb_camera_link_frame">
     </link>
-    <joint name="${sensor_name}_camera_frame_joint" type="fixed">
-        <origin xyz="${camera_box_x} 0 0" rpy="0 0 0" />
-        <parent link="${sensor_name}_camera_link" />
-        <child link="${sensor_name}_camera_link_frame" />
+    <joint name="${robot_name}_rgb_camera_link_frame_joint" type="fixed">
+        <origin rpy="${camera_ROLL} ${camera_PITCH} ${camera_YAW}" xyz="${origin_xyz}"/>
+        <parent link="${parent_name}" />
+        <child link="${robot_name}_rgb_camera_link_frame" />
         <axis xyz="0 0 0"/>
     </joint>
-    <gazebo reference="${sensor_name}_camera_link_frame">
-          <sensor type="camera" name="${sensor_name}">
-            <always_on>1</always_on>
-            <update_rate>1</update_rate>
-            <camera name="head">
-                <horizontal_fov>1.3962634</horizontal_fov>
-                <image>
-                <width>300</width>
-                <height>300</height>
-                <format>R8G8B8</format>
-                </image>
-                <clip>
-                <near>0.02</near>
-                <far>20.0</far>
-                </clip>
-                <noise>
-                <type>gaussian</type>
-                <!-- Noise is sampled independently per pixel on each frame.
-                    That pixel's noise value is added to each of its color
-                    channels, which at that point lie in the range [0,1]. -->
-                <mean>0.0</mean>
-                <stddev>0.007</stddev>
-                </noise>
-                <always_on>1</always_on>
-                <update_rate>30</update_rate>
-            </camera>
-            <plugin name="plugin_name" filename="libgazebo_ros_camera.so">
-                <ros>
-                <namespace>${sensor_name}_ns</namespace>
-                <argument>image_raw:=${sensor_name}_img</argument>
-                <argument>camera_info:=${sensor_name}_info</argument>
-                </ros>
-                <camera_name>${sensor_name}_camera</camera_name>
-                <frame_name>${sensor_name}_camera_link_frame</frame_name>
-                <hack_baseline>0.07</hack_baseline>
-            </plugin>
-        </sensor>
-    </gazebo>
-  </xacro:macro>
-  <xacro:macro name="wide_angle_camera" params="parent_name sensor_name origin_xyz camera_YAW">
-    <link name='${sensor_name}_camera_link'>
-		<visual>
-			<origin xyz="0 0 0"
-					rpy="0 0 0"/>
-			<geometry>
-				<box size="${camera_box_x} ${camera_box_y} ${camera_box_z}"/>
-			</geometry>
-		</visual>
-	</link>
-    <joint name="${sensor_name}_camera_link_joint" type="fixed">
-		<origin rpy="0 0 ${camera_YAW}" xyz="${origin_xyz}"/>
-		<parent link="${parent_name}"/>
-		<child link="${sensor_name}_camera_link"/>
-	</joint>
-    <link name="${sensor_name}_camera_link_frame">
-    </link>
-    <joint name="${sensor_name}_camera_frame_joint" type="fixed">
-        <origin xyz="${camera_box_x} 0 0" rpy="0 0 0" />
-        <parent link="${sensor_name}_camera_link" />
-        <child link="${sensor_name}_camera_link_frame" />
-        <axis xyz="0 0 0"/>
-    </joint>
-    <gazebo reference="${sensor_name}_camera_link_frame">
+    <gazebo reference="${robot_name}_rgb_camera_link_frame">
         <sensor name="camera" type="wideanglecamera">
           <camera>
@@ -127,8 +50,11 @@
           </camera>
           <plugin name="camera_controller" filename="libgazebo_ros_camera.so">
-            <cameraName>${sensor_name}</cameraName>
+            <ros>
+              <namespace>/${robot_name}</namespace>
+            </ros>
+            <cameraName>rgb_camera</cameraName>
             <imageTopicName>image_raw</imageTopicName>
             <cameraInfoTopicName>camera_info</cameraInfoTopicName>
-            <frameName>${sensor_name}_camera_link_frame</frameName>
+            <frameName>${robot_name}_rgb_camera_link_frame</frameName>
             <hackBaseline>0.07</hackBaseline>
           </plugin>
@@ -136,78 +62,52 @@
     </gazebo>
   </xacro:macro>
-  <xacro:macro name="laser_scan" params="parent_name sensor_name origin_xyz sensor_YAW">
-    <link name='${sensor_name}_laser_scan_link'>
-        <visual name="visual_${parent_name}">
-            <geometry>
-                    <mesh filename="package://box_bot_description/meshes/sensors/rplidar.dae" scale="1.0 1.0 1.0"/>
-            </geometry>
-        </visual>
+  <xacro:macro name="laser_scan" params="robot_name parent_name origin_xyz sensor_YAW">
+    <link name="${robot_name}_laser_scan_frame">
+    </link>
+    <joint name="${robot_name}_laser_scan_frame_joint" type="fixed">
+        <origin xyz="${origin_xyz}" rpy="0 0 ${sensor_YAW}" />
+        <parent link="${parent_name}" />
+        <child link="${robot_name}_laser_scan_frame" />
+    </joint>
+    <gazebo reference="${robot_name}_laser_scan_frame">
+      <sensor name="sensor_ray" type="ray">
+          <pose>0 0 0 0 0 0</pose>
+          <ray>
+            <scan>
+              <horizontal>
+                <samples>200</samples>
+                <resolution>1.0</resolution>
+                <min_angle>-3.14</min_angle>
+                <max_angle>3.14</max_angle>
+              </horizontal>
+            </scan>
+            <range>
+              <min>0.1</min>
+              <max>5.0</max>
+            </range>
+          </ray>
+          <always_on>true</always_on>
+          <visualize>true</visualize>
+          <update_rate>100.0</update_rate>
+          <plugin name="laser" filename="libgazebo_ros_ray_sensor.so">
+            <ros>
+              <namespace>/${robot_name}</namespace>
+              <remapping>~/out:=laser_scan</remapping>
+            </ros>
+            <output_type>sensor_msgs/LaserScan</output_type>
+          </plugin>
+        </sensor>
+    </gazebo>
+  </xacro:macro>
+<xacro:macro name="point_cloud_sensor" params="robot_name parent_name sensor_name origin_xyz sensor_YAW">
+  <link name='${robot_name}_pointcloud_link'>
 	</link>
-    <joint name="${sensor_name}_laser_scan_link_joint" type="fixed">
-		<origin rpy="0 0 ${sensor_YAW - 1.5708}" xyz="${origin_xyz}"/>
+  <joint name="${robot_name}_pointcloud_link_joint" type="fixed">
+		<origin rpy="0 0 ${sensor_YAW}" xyz="${origin_xyz}"/>
 		<parent link="${parent_name}"/>
-		<child link="${sensor_name}_laser_scan_link"/>
+		<child link="${robot_name}_pointcloud_link"/>
 	</joint>
-    <link name="${sensor_name}_laser_scan_frame">
-    </link>
-    <joint name="${sensor_name}_laser_scan_frame_joint" type="fixed">
-        <origin xyz="0 0 0.03" rpy="0 0 0" />
-        <parent link="${sensor_name}_laser_scan_link" />
-        <child link="${sensor_name}_laser_scan_frame" />
-        <axis xyz="0 0 0"/>
-    </joint>
-	<gazebo reference="${sensor_name}_laser_scan_frame">
-		<sensor name="sensor_ray" type="ray">
-        <pose>0 0 0 0 0 0</pose>
-        <ray>
-          <scan>
-            <horizontal>
-              <samples>200</samples>
-              <resolution>1.0</resolution>
-              <min_angle>-1.0</min_angle>
-              <max_angle>1.0</max_angle>
-            </horizontal>
-          </scan>
-          <range>
-            <min>0.05</min>
-            <max>10.0</max>
-          </range>
-        </ray>
-        <always_on>true</always_on>
-        <visualize>true</visualize>
-        <update_rate>100.0</update_rate>
-        <plugin name="laser" filename="libgazebo_ros_ray_sensor.so">
-          <ros>
-            <namespace>/box_bot</namespace>
-            <remapping>~/out:=laser_scan</remapping>
-          </ros>
-          <output_type>sensor_msgs/LaserScan</output_type>
-        </plugin>
-      </sensor>
-	</gazebo>
-  </xacro:macro>
-<xacro:macro name="block_laser_scan" params="parent_name sensor_name origin_xyz sensor_YAW">
-    <link name='${sensor_name}_laser_scan_link'>
-        <visual name="visual_${parent_name}">
-            <geometry>
-                    <mesh filename="package://box_bot_description/meshes/sensors/realsense.dae" scale="0.25 0.25 0.25"/>
-            </geometry>
-        </visual>
-	</link>
-    <joint name="${sensor_name}_laser_scan_link_joint" type="fixed">
-		<origin rpy="0 0 ${sensor_YAW - 1.5708}" xyz="${origin_xyz}"/>
-		<parent link="${parent_name}"/>
-		<child link="${sensor_name}_laser_scan_link"/>
-	</joint>
-    <link name="${sensor_name}_laser_scan_frame">
-    </link>
-    <joint name="${sensor_name}_laser_scan_frame_joint" type="fixed">
-        <origin xyz="0 0 0" rpy="0 0 0" />
-        <parent link="${sensor_name}_laser_scan_link" />
-        <child link="${sensor_name}_laser_scan_frame" />
-        <axis xyz="0 0 0"/>
-    </joint>
-    <gazebo reference="${sensor_name}_laser_scan_frame">
-        <sensor type="ray" name="block_laser_sensor">
+    <gazebo reference="${robot_name}_pointcloud_link">
+        <sensor type="ray" name="pointcloud_sensor">
             <ray>
             <scan>
@@ -242,10 +142,10 @@
             <!-- Change namespace and output topic so published topic is /rrbot/laser/pointcloud -->
             <ros>
-                <namespace>/rrbot/laser</namespace>
+                <namespace>/${robot_name}/pointcloud</namespace>
                 <argument>~/out:=pointcloud</argument>
             </ros>
             <!-- Set output to sensor_msgs/PointCloud to get same output type as gazebo_ros_block_laser -->
             <output_type>sensor_msgs/PointCloud</output_type>
-            <!-- <frame_name> ommited, will default to block_laser_link -->
+            <frameName>${robot_name}_pointcloud_link</frameName>
             <!-- min_intensity instead of hokuyoMinIntensity -->
             <min_intensity>100.0</min_intensity>

File: box_bot_description/robot/wheels.xacro (robot description, xacro)
@@ -2,6 +2,6 @@
 <robot xmlns:xacro="http://www.ros.org/wiki/xacro">
     <!-- Wheels-->
-    <xacro:macro  name="link_wheel" params="name r l incr">
-      <link name="${name}">
+    <xacro:macro  name="wheel" params="parent child origin_xyz robot_name name_wheel_link r l incr">
+      <link name="${robot_name}_${name_wheel_link}">
           <inertial>
             <mass value="0.2"/>
@@ -9,5 +9,5 @@
               <xacro:cylinder_inertia mass="0.2" r="${r}" l="${l}" />
           </inertial>
-          <collision name="${name}_collision">
+          <collision name="${robot_name}_${name_wheel_link}_collision">
             <origin rpy="0 1.5707 1.5707" xyz="0 0 0"/>
             <geometry>
@@ -15,5 +15,5 @@
             </geometry>
           </collision>
-          <visual name="${name}_visual">
+          <visual name="${robot_name}_${name_wheel_link}_visual">
             <origin rpy="0 1.5707 1.5707" xyz="0 0 0"/>
             <geometry>
@@ -22,5 +22,5 @@
           </visual>
       </link>
-      <gazebo reference="${name}">
+      <gazebo reference="${robot_name}_${name_wheel_link}">
         <kp>${kp_wheel}</kp>
         <kd>${kd_wheel}</kd>
@@ -29,14 +29,12 @@
         <material>Gazebo/White</material>
       </gazebo>
-  </xacro:macro >
-  <xacro:macro  name="joint_wheel" params="name parent child origin_xyz">
-    <joint name="${name}" type="continuous">
-      <origin rpy="0 0 0" xyz="${origin_xyz}"/>
-      <child link="${child}"/>
-      <parent link="${parent}"/>
-      <axis rpy="0 0 0" xyz="0 1 0"/>
-      <limit effort="10000" velocity="1000"/>
-      <joint_properties damping="1.0" friction="1.0"/>
-    </joint>
+      <joint name="${robot_name}_${name_wheel_link}_joint" type="continuous">
+        <origin rpy="0 0 0" xyz="${origin_xyz}"/>
+        <child link="${child}"/>
+        <parent link="${parent}"/>
+        <axis rpy="0 0 0" xyz="0 1 0"/>
+        <limit effort="10000" velocity="1000"/>
+        <joint_properties damping="1.0" friction="1.0"/>
+      </joint>
   </xacro:macro >
 </robot>

Commit message: Added mods and upgrades to be able to use rmf better

File: box_bot_description/robot/box_bot.xacro (robot description, xacro)
@@ -11,11 +11,13 @@
   <xacro:arg name="box_bot_name" default="box_bot"/>
   <xacro:box_bot_body robot_name="$(arg box_bot_name)"/>
-  <xacro:wheel parent="$(arg box_bot_name)_chassis" child="$(arg box_bot_name)_right_wheel" origin_xyz="0 ${base_box_x / 2.0} ${-1.0 * wheel_radius}" robot_name="$(arg box_bot_name)" name_wheel_link="right_wheel" r="${wheel_radius}" l="${wheel_width}" incr="${wheel_increment}"/>
-  <xacro:wheel parent="$(arg box_bot_name)_chassis" child="$(arg box_bot_name)_left_wheel" origin_xyz="0 ${-1.0 * base_box_x / 2.0} ${-1.0 * wheel_radius}" robot_name="$(arg box_bot_name)" name_wheel_link="left_wheel" r="${wheel_radius}" l="${wheel_width}" incr="${wheel_increment}"/>
+  <xacro:wheel parent="$(arg box_bot_name)_chassis" child="$(arg box_bot_name)_right_wheel" origin_xyz="0 ${-1.0 * base_box_x / 2.0} ${-1.0 * wheel_radius}" robot_name="$(arg box_bot_name)" name_wheel_link="right_wheel" r="${wheel_radius}" l="${wheel_width}" incr="${wheel_increment}"/>
+  <xacro:wheel parent="$(arg box_bot_name)_chassis" child="$(arg box_bot_name)_left_wheel" origin_xyz="0 ${base_box_x / 2.0} ${-1.0 * wheel_radius}" robot_name="$(arg box_bot_name)" name_wheel_link="left_wheel" r="${wheel_radius}" l="${wheel_width}" incr="${wheel_increment}"/>
   <xacro:caster_wheel robot_name="$(arg box_bot_name)" parent="$(arg box_bot_name)_chassis" caster_wheel_name="front" origin_xyz="${(base_box_x / 2.0) - wheel_increment} 0 ${-1.0* base_box_x / 2.0}" radius="${wheel_increment}" legth="${dummy_length}"/>
   <xacro:caster_wheel robot_name="$(arg box_bot_name)" parent="$(arg box_bot_name)_chassis" caster_wheel_name="back" origin_xyz="${(-1.0 *base_box_x / 2.0) + wheel_increment} 0 ${-1.0* base_box_x / 2.0}" radius="${wheel_increment}" legth="${dummy_length}"/>
   <xacro:box_bot_gazebo_systems robot_name="$(arg box_bot_name)"/>
+<!--
   <xacro:laser_scan robot_name="$(arg box_bot_name)" parent_name="$(arg box_bot_name)_chassis" origin_xyz="0.0 0.0 ${base_box_x / 2.0}" sensor_YAW="0.0"/>
   <xacro:point_cloud_sensor robot_name="$(arg box_bot_name)" parent_name="$(arg box_bot_name)_chassis" sensor_name="block_laser_scan" origin_xyz="${base_box_x/ 1.9} 0.0 0.0" sensor_YAW="0.0"/>
+   -->
   <xacro:camera_rgb robot_name="$(arg box_bot_name)" parent_name="$(arg box_bot_name)_chassis" origin_xyz="${base_box_x/ 1.9} 0.0 ${base_box_x / 2.0}" camera_ROLL="0.0" camera_PITCH="0.0" camera_YAW="0.0"/>
 </robot>

File: box_bot_description/robot/box_bot_body.xacro (robot description, xacro)
@@ -7,5 +7,5 @@
         <visual>
           <geometry>
-            <mesh filename="package://box_bot_description/meshes/box_bot_1.dae" scale="0.1 0.1 0.1"/>
+            <mesh filename="package://box_bot_description/meshes/${robot_name}.dae" scale="0.1 0.1 0.1"/>
           </geometry>
         </visual>

File: box_bot_description/robot/box_bot_slotcar.xacro (robot description, xacro)
@@ -11,10 +11,11 @@
   <xacro:arg name="box_bot_name" default="box_bot_1"/>
   <xacro:box_bot_body robot_name="$(arg box_bot_name)"/>
-  <xacro:wheel parent="$(arg box_bot_name)_chassis" child="$(arg box_bot_name)_left_wheel" origin_xyz="0 ${base_box_x / 2.0} ${-1.0 * wheel_radius}" robot_name="$(arg box_bot_name)" name_wheel_link="left" r="${wheel_radius}" l="${wheel_width}" incr="${wheel_increment}"/>
-  <xacro:wheel parent="$(arg box_bot_name)_chassis" child="$(arg box_bot_name)_right_wheel" origin_xyz="0 ${-1.0 * base_box_x / 2.0} ${-1.0 * wheel_radius}" robot_name="$(arg box_bot_name)" name_wheel_link="right" r="${wheel_radius}" l="${wheel_width}" incr="${wheel_increment}"/>
+  <xacro:wheel parent="$(arg box_bot_name)_chassis" child="$(arg box_bot_name)_right_wheel" origin_xyz="0 ${-1.0 * base_box_x / 2.0} ${-1.0 * wheel_radius}" robot_name="$(arg box_bot_name)" name_wheel_link="right_wheel" r="${wheel_radius}" l="${wheel_width}" incr="${wheel_increment}"/>
+  <xacro:wheel parent="$(arg box_bot_name)_chassis" child="$(arg box_bot_name)_left_wheel" origin_xyz="0 ${base_box_x / 2.0} ${-1.0 * wheel_radius}" robot_name="$(arg box_bot_name)" name_wheel_link="left_wheel" r="${wheel_radius}" l="${wheel_width}" incr="${wheel_increment}"/>
   <xacro:caster_wheel robot_name="$(arg box_bot_name)" parent="$(arg box_bot_name)_chassis" caster_wheel_name="front" origin_xyz="${(base_box_x / 2.0) - wheel_increment} 0 ${-1.0* base_box_x / 2.0}" radius="${wheel_increment}" legth="${dummy_length}"/>
   <xacro:caster_wheel robot_name="$(arg box_bot_name)" parent="$(arg box_bot_name)_chassis" caster_wheel_name="back" origin_xyz="${(-1.0 *base_box_x / 2.0) + wheel_increment} 0 ${-1.0* base_box_x / 2.0}" radius="${wheel_increment}" legth="${dummy_length}"/>
-  <xacro:box_bot_gazebo_systems_slotcar robot_name="$(arg box_bot_name)"/>
-  <!-- <xacro:laser_scan robot_name="$(arg box_bot_name)" parent_name="$(arg box_bot_name)_chassis" origin_xyz="0.0 0.0 ${base_box_x / 2.0}" sensor_YAW="0.0"/>
+  <xacro:box_bot_gazebo_systems_slotcar robot_name="$(arg box_bot_name)" name_left_wheel_link="left_wheel" name_right_wheel_link="right_wheel"/>
+<!--
+  <xacro:laser_scan robot_name="$(arg box_bot_name)" parent_name="$(arg box_bot_name)_chassis" origin_xyz="0.0 0.0 ${base_box_x / 2.0}" sensor_YAW="0.0"/>
   <xacro:point_cloud_sensor robot_name="$(arg box_bot_name)" parent_name="$(arg box_bot_name)_chassis" sensor_name="block_laser_scan" origin_xyz="${base_box_x/ 1.9} 0.0 0.0" sensor_YAW="0.0"/>
    -->

File: box_bot_description/robot/wheels.xacro (robot description, xacro)
@@ -29,5 +29,6 @@
         <material>Gazebo/White</material>
       </gazebo>
-      <joint name="${robot_name}/joint_tire_${name_wheel_link}" type="continuous">
+        box_bot_3_left_wheel_joint
+      <joint name="${robot_name}_${name_wheel_link}_joint" type="continuous">
         <origin rpy="0 0 0" xyz="${origin_xyz}"/>
         <child link="${robot_name}_${name_wheel_link}"/>
