Commit message: drift attempts

File: robot_description/robot/parts/omni_wheel/omni_wheel.xacro (robot description, xacro)
@@ -9,4 +9,5 @@
           <limit effort="100" velocity="100"/>
 	  <xacro:insert_block name="joint_axis"/>
+    <!-- <dynamics damping="0.001" friction="0.001"/> -->
 	</joint>
 	<link name="${prefix}_wheel_link">

File: robot_description/robot/parts/roller/roller.xacro (robot description, xacro)
@@ -8,4 +8,5 @@
 	  <child link="${prefix}_roller_link"/>
 	  <xacro:insert_block name="joint_axis"/>
+	  <!-- <dynamics damping="0.0" friction="0.001"/> -->
 	</joint>
 	<link name="${prefix}_roller_link">
